File: hardware/powermod.kicad_sch (KiCad schematic)
At the start: 73 parts, among them J1 USB_C_IN, J2 USB_C_OUT, J3 JST_PH_2, J4 STEMMA_QT, J5 SWD_HDR, Q1 AON7407, Q2 AON7407, Q3 BSS138, SW1 BUTTON, U1 BM8563ESA, U2 PY32F003F18P6, U3 TPS63020DSJR, U4 TP4056, U5 XC6206P332MR, Y1 Q13FC13500004

Commit message: hardware: CORRECT USB-C CC pins -> A5/B5 (revert a2826a7) + full reroute
Deep pre-fab audit found the USB-C CC assignment was WRONG: a2826a7 moved CC to
A8/B8 (the SBU pins) on a false "mirrored footprint" claim. Verified 3 ways that
A5=CC1/B5=CC2 and A8/B8=SBU: (1) USB-C spec; (2) real C165948 = TYPE-C-31-M-12
standard pinout (LCSC/EasyEDA land pattern); (3) KiCad's HRO TYPE-C-31-M-12
footprint is geometrically identical to ours (A5@-1.25=CC1, A8@+1.25=SBU1). With
CC on A8/B8 the Rp/Rd resistors sat on floating SBU pins -> board would never
negotiate VBUS.

Fix: netlist CC back to A5/B5, A8/B8->NC. R4/R5 CC labels swapped (symmetric 56k)
so each Rp stays beside its pad after the move. Board pads reassigned to match;
full Freerouting reroute. pad-diff 226/226, CC verified on A5/B5, DRC 0 shorts.

Remaining hand-finish (this seed): 4 track_width (L1N/L2 necks), and unrouted =
J1/J2 VBUS/VOUT escapes + CC2_IN(B5) + R5.2(VOUT) + TP3. EP got 1 GND tie this
run (In2 SCL crowds it).

Co-Authored-By: Claude Opus 4.8 <noreply@anthropic.com>
Connections:
- net CC1_OUT: now also R5.1; no longer R4.1
- net CC2_OUT: now also R4.1; no longer R5.1
- no-connect marks 11 -> 15
Changed lines of the file:
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@@
   (pin "A5")
   (pin "B5")
+  (pin "A8")
+  (pin "B8")
   (pin "A6")
   (pin "A7")
@@
   (pin "A5")
   (pin "B5")
+  (pin "A8")
+  (pin "B8")
   (pin "A6")
   (pin "A7")
@@
  (global_label "CHG_JPD" (shape passive) (at 166.37 426.72 0) (effects (font (size 1.0 1.0)) (justify left)))
  (global_label "CHG_JP" (shape passive) (at 179.07 426.72 0) (effects (font (size 1.0 1.0)) (justify left)))
- (global_label "GND" (shape passive) (at 234.95 24.130000000000003 0) (effects (font (size 1.0 1.0)) (justify left)))
- (global_label "GND" (shape passive) (at 234.95 26.67 0) (effects (font (size 1.0 1.0)) (justify left)))
- (global_label "VBUS" (shape passive) (at 234.95 29.21 0) (effects (font (size 1.0 1.0)) (justify left)))
- (global_label "VBUS" (shape passive) (at 234.95 31.75 0) (effects (font (size 1.0 1.0)) (justify left)))
- (global_label "CC1_IN" (shape passive) (at 234.95 34.29 0) (effects (font (size 1.0 1.0)) (justify left)))
- (global_label "CC2_IN" (shape passive) (at 234.95 36.83 0) (effects (font (size 1.0 1.0)) (justify left)))
- (global_label "GND" (shape passive) (at 252.73000000000002 34.29 0) (effects (font (size 1.0 1.0)) (justify left)))
- (global_label "GND" (shape passive) (at 234.95 90.17000000000002 0) (effects (font (size 1.0 1.0)) (justify left)))
- (global_label "GND" (shape passive) (at 234.95 92.71000000000001 0) (effects (font (size 1.0 1.0)) (justify left)))
- (global_label "VOUT" (shape passive) (at 234.95 95.25000000000001 0) (effects (font (size 1.0 1.0)) (justify left)))
- (global_label "VOUT" (shape passive) (at 234.95 97.79 0) (effects (font (size 1.0 1.0)) (justify left)))
- (global_label "CC1_OUT" (shape passive) (at 234.95 100.33000000000001 0) (effects (font (size 1.0 1.0)) (justify left)))
- (global_label "CC2_OUT" (shape passive) (at 234.95 102.87 0) (effects (font (size 1.0 1.0)) (justify left)))
- (global_label "GND" (shape passive) (at 252.73000000000002 100.33000000000001 0) (effects (font (size 1.0 1.0)) (justify left)))
+ (global_label "GND" (shape passive) (at 234.95 22.86 0) (effects (font (size 1.0 1.0)) (justify left)))
+ (global_label "GND" (shape passive) (at 234.95 25.4 0) (effects (font (size 1.0 1.0)) (justify left)))
+ (global_label "VBUS" (shape passive) (at 234.95 27.94 0) (effects (font (size 1.0 1.0)) (justify left)))
+ (global_label "VBUS" (shape passive) (at 234.95 30.48 0) (effects (font (size 1.0 1.0)) (justify left)))
+ (global_label "CC1_IN" (shape passive) (at 234.95 33.02 0) (effects (font (size 1.0 1.0)) (justify left)))
+ (global_label "CC2_IN" (shape passive) (at 234.95 35.56 0) (effects (font (size 1.0 1.0)) (justify left)))
+ (global_label "GND" (shape passive) (at 252.73000000000002 35.56 0) (effects (font (size 1.0 1.0)) (justify left)))
+ (global_label "GND" (shape passive) (at 234.95 88.9 0) (effects (font (size 1.0 1.0)) (justify left)))
+ (global_label "GND" (shape passive) (at 234.95 91.44000000000001 0) (effects (font (size 1.0 1.0)) (justify left)))
+ (global_label "VOUT" (shape passive) (at 234.95 93.98 0) (effects (font (size 1.0 1.0)) (justify left)))
+ (global_label "VOUT" (shape passive) (at 234.95 96.52000000000001 0) (effects (font (size 1.0 1.0)) (justify left)))
+ (global_label "CC1_OUT" (shape passive) (at 234.95 99.06000000000002 0) (effects (font (size 1.0 1.0)) (justify left)))
+ (global_label "CC2_OUT" (shape passive) (at 234.95 101.60000000000001 0) (effects (font (size 1.0 1.0)) (justify left)))
+ (global_label "GND" (shape passive) (at 252.73000000000002 101.60000000000001 0) (effects (font (size 1.0 1.0)) (justify left)))
  (global_label "VBAT" (shape passive) (at 237.49 162.56 0) (effects (font (size 1.0 1.0)) (justify left)))
  (global_label "GND" (shape passive) (at 250.19 162.56 0) (effects (font (size 1.0 1.0)) (justify left)))
@@
  (global_label "CC2_IN" (shape passive) (at 521.97 294.64000000000004 0) (effects (font (size 1.0 1.0)) (justify left)))
  (global_label "GND" (shape passive) (at 534.6700000000001 294.64000000000004 0) (effects (font (size 1.0 1.0)) (justify left)))
- (global_label "CC1_OUT" (shape passive) (at 521.97 360.68000000000006 0) (effects (font (size 1.0 1.0)) (justify left)))
+ (global_label "CC2_OUT" (shape passive) (at 521.97 360.68000000000006 0) (effects (font (size 1.0 1.0)) (justify left)))
  (global_label "VOUT" (shape passive) (at 534.6700000000001 360.68000000000006 0) (effects (font (size 1.0 1.0)) (justify left)))
- (global_label "CC2_OUT" (shape passive) (at 521.97 426.72 0) (effects (font (size 1.0 1.0)) (justify left)))
+ (global_label "CC1_OUT" (shape passive) (at 521.97 426.72 0) (effects (font (size 1.0 1.0)) (justify left)))
  (global_label "VOUT" (shape passive) (at 534.6700000000001 426.72 0) (effects (font (size 1.0 1.0)) (justify left)))
  (global_label "VBAT" (shape passive) (at 593.09 30.48 0) (effects (font (size 1.0 1.0)) (justify left)))
@@
  (global_label "OSCI" (shape passive) (at 735.33 162.56 0) (effects (font (size 1.0 1.0)) (justify left)))
  (global_label "OSCO" (shape passive) (at 748.0300000000001 162.56 0) (effects (font (size 1.0 1.0)) (justify left)))
- (no_connect (at 252.73000000000002 24.130000000000003))
- (no_connect (at 252.73000000000002 26.67))
- (no_connect (at 252.73000000000002 29.21))
- (no_connect (at 252.73000000000002 31.75))
- (no_connect (at 252.73000000000002 90.17000000000002))
- (no_connect (at 252.73000000000002 92.71000000000001))
- (no_connect (at 252.73000000000002 95.25000000000001))
- (no_connect (at 252.73000000000002 97.79))
+ (no_connect (at 234.95 38.1))
+ (no_connect (at 252.73000000000002 22.86))
+ (no_connect (at 252.73000000000002 25.4))
+ (no_connect (at 252.73000000000002 27.94))
+ (no_connect (at 252.73000000000002 30.48))
+ (no_connect (at 252.73000000000002 33.02))
+ (no_connect (at 234.95 104.14000000000001))
+ (no_connect (at 252.73000000000002 88.9))
+ (no_connect (at 252.73000000000002 91.44000000000001))
+ (no_connect (at 252.73000000000002 93.98))
+ (no_connect (at 252.73000000000002 96.52000000000001))
+ (no_connect (at 252.73000000000002 99.06000000000002))
  (no_connect (at 234.95 229.87))
  (no_connect (at 679.45 295.91))
